Commit message: Save Lite3 perception, dynamic avoidance and bug-fix history
Preserve the complete six-package workspace, 3D lidar processing, unified
bringup, terminal and Gazebo goal interfaces, MPPI avoidance and recovery,
Lattice footprint planning, reverse manoeuvres and final-approach fallback.

Document the observed failures, diagnosis, fixes, retained limitations and
Gazebo/protocol evidence. Refresh the project introduction, recovery guide,
progress report, full inventory and SHA256 manifest; archive older summaries.

Keep pretrained policy recovery snapshots and licenses, original architecture
and roadmap, and exclude generated outputs, caches and credentials.

File: src/lite3_description/urdf/Lite3_gazebo.urdf (robot description, URDF)
Before this commit: robot Lite3, 17 links, 16 joints
Links:
- added link lidar_link; visual cylinder length=0.03 radius=0.035
Joints:
- added joint lidar_mount: type fixed, parent TORSO, child lidar_link, origin xyz=0.30 0 0.15 rpy=0 0 0
